File: H40R00/Design/H40R00.brd (EAGLE design)
At the start: 34.6 x 30 mm, 36 parts, among them P1 HEXABIT_17.32_NO_P3, U1 STLINK-V3MODS

Commit message: Finished placement and routing
Parts:
- removed C, D, R: PAD1, HEXABITZ_CONNECTION_PARTS:PAD1
- removed CAN_RX, CAN_TX, CLK, CTS, DIR, IO0, IO1, IO2, IO3, MISO, MOSI, NSS, RTS, RX, SCL, SDA, SWO, TX: PAD4, HEXABITZ_CONNECTION_PARTS:PAD4
- removed JP10, JP2, JP3, JP4, JP5, JP6, JP7, JP8, JP9: (no value), jumper:JP1
- added VRX, VTX: PAD4, HEXABITZ_CONNECTION_PARTS:PAD4
- added VRX1, VRX2, VRX3, VRX4, VTX1, VTX2, VTX3, VTX4: (no value), jumper:SJ
- JP1: device jumper:JP1 -> pinhead:1X02
- P1: value HEXABIT_17.32_NO_P3 -> HEXABIT_17.32_NO_P3_P6_P7_P12; device hexabitz_connectors:HEXABIT_17.32_NO_P3 -> hexabitz_connectors:HEXABIT_17.32_NO_P3_P6_P7_P12
- SWD: device con-lsta:FE05-1 -> con-lstb:MA03-1
- moved SWD 244.8 mm to (45.2, 34.7), turned to 90 degrees
- moved R2 228.3 mm to (38.5, 48.1), flipped to the bottom
- moved R1 223.3 mm to (30.9, 48.1), flipped to the bottom, turned to 180 degrees
- moved JP1 211.2 mm to (24.1, 34.7), turned to 90 degrees
- moved U1 42.1 mm to (34.6, 19.7), turned to 180 degrees
- moved P1 0.07 mm to (34.7, 34.7)
Connections:
- removed net N$11: CAN_RX.P$1, U1.9
- removed net N$12: CAN_TX.P$1, U1.10
- removed net N$14: MISO.P$1, U1.23
- removed net N$15: MOSI.P$1, U1.25
- removed net N$16: NSS.P$1, U1.14
- removed net N$17: CLK.P$1, U1.7
- removed net N$18: IO0.P$1, U1.18
- removed net N$19: IO1.P$1, U1.19
- removed net N$20: IO2.P$1, U1.20
- removed net N$21: IO3.P$1, U1.21
- removed net N$4: SWO.P$1, U1.6
- removed net N$5: DIR.P$1, U1.32
- removed net N$6: RX.P$1, U1.1
- removed net N$7: CTS.P$1, U1.2
- removed net N$8: RTS.P$1, U1.3
- removed net N$9: TX.P$1, U1.11
- removed net UART5_RX: JP10.2, P1.PAD_PD6
- removed net UART5_TX: JP5.2, P1.PAD_PU6
- net GND: now also JP1.1; no longer P1.PAD_PD12, P1.PAD_PD7, SWD.1
- net N$10: no longer SCL.P$1
- net N$13: no longer SDA.P$1
- net SWD_C: now also SWD.2; no longer C.P$1, C.P$2, SWD.4
- net SWD_D: now also SWD.1; no longer D.P$1, D.P$2, SWD.3
- net SWD_R: now also SWD.3; no longer R.P$1, R.P$2, SWD.5
- net UART2_RX: now also VRX1.1; no longer JP6.2
- net UART2_TX: now also VTX1.1; no longer JP1.2
- net UART3_RX: now also VRX3.1; no longer JP8.2
- net UART3_TX: now also VTX3.1; no longer JP3.2
- net UART4_RX: now also VRX4.1; no longer JP9.2
- net UART4_TX: now also VTX4.1; no longer JP4.2
- net UART6_RX: now also VRX2.1; no longer JP7.2
- net UART6_TX: now also VTX2.1; no longer JP2.2
- net VCP_RX: now also VRX.P$1, VRX1.2, VRX2.2, VRX3.2, VRX4.2; no longer JP10.1
- net VCP_TX: now also VTX.P$1, VTX1.2, VTX2.2, VTX3.2, VTX4.2; no longer JP1.1, JP2.1, JP3.1, JP4.1, JP5.1
- net VDD: now also JP1.2; no longer P1.PAD_PU12, P1.PAD_PU7, SWD.2
Routing:
- net VCP_TX: track 0.00 -> 42.8 mm, vias 0 -> 4
- net VCP_RX: track 0.00 -> 39.8 mm, vias 0 -> 1
- net SWD_R: track 0.00 -> 22.5 mm, vias 0 -> 1
- net GND: track 0.05 -> 21.4 mm, vias 5 -> 7
- net UART4_TX: track 28.3 -> 8.94 mm
- net UART4_RX: track 24.3 -> 9.29 mm, vias 2 -> 0
- net SWD_C: track 0.00 -> 13.8 mm
- net UART6_RX: track 20.8 -> 8.75 mm, vias 2 -> 0
- net UART3_RX: track 18.4 -> 8.94 mm
- net UART2_RX: track 18.1 -> 9.42 mm
- net UART3_TX: track 17.1 -> 9.55 mm
- net UART2_TX: track 18.1 -> 11.9 mm
- net VDD: track 0.00 -> 5.92 mm, vias 0 -> 1
- net UART5_TX: track 4.72 -> 0.00 mm, vias 1 -> 0
- net SWD_D: track 0.00 -> 3.79 mm
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- removed copper zone on layer 1, net GND
Other:
- board text added: "1"
- board text added: "32"
- board text added: "H40R00"
- board text removed: "B"
- board text removed: "H1AR10"
- board text removed: "P5"

Commit message: Generate output files Release V0
Parts:
- R1, R2: value (none) -> 680
Changed lines of the file:
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@@
 <attribute name="VENDOR" value="STMicroelectronics" x="34.625025" y="19.685" locked="yes" size="1.778" layer="27" rot="R180" display="off"/>
 </element>
-<element name="R1" library="HEXABITZ_RCLS" library_urn="urn:adsk.eagle:library:20064561" package="R-0603" package3d_urn="urn:adsk.eagle:package:1435818/3" value="" x="30.861" y="48.133" smashed="yes" rot="MR180">
+<element name="R1" library="HEXABITZ_RCLS" library_urn="urn:adsk.eagle:library:20064561" package="R-0603" package3d_urn="urn:adsk.eagle:package:1435818/3" value="680" x="30.861" y="48.133" smashed="yes" rot="MR180">
 <attribute name="MFN" value="Yageo" x="30.861" y="48.133" size="1.778" layer="28" rot="MR180" display="off"/>
 <attribute name="MPN" value="RC0603JR-07680RL" x="30.861" y="48.133" size="1.778" layer="28" rot="MR180" display="off"/>
@@
 <attribute name="VALUE" x="30.226" y="50.038" size="1.27" layer="28" rot="MR180"/>
 </element>
-<element name="R2" library="HEXABITZ_RCLS" library_urn="urn:adsk.eagle:library:20064561" package="R-0603" package3d_urn="urn:adsk.eagle:package:1435818/3" value="" x="38.481" y="48.133" smashed="yes" rot="MR0">
+<element name="R2" library="HEXABITZ_RCLS" library_urn="urn:adsk.eagle:library:20064561" package="R-0603" package3d_urn="urn:adsk.eagle:package:1435818/3" value="680" x="38.481" y="48.133" smashed="yes" rot="MR0">
 <attribute name="MFN" value="Yageo" x="38.481" y="48.133" size="1.778" layer="28" rot="MR0" display="off"/>
 <attribute name="MPN" value="RC0603JR-07680RL" x="38.481" y="48.133" size="1.778" layer="28" rot="MR0" display="off"/>
