File: H40R00/Design/H40R00.sch (EAGLE design)
At the start: 36 parts, among them P1 HEXABIT_17.32_NO_P3, U1 STLINK-V3MODS

Commit message: Finished placement and routing
Parts:
- removed C, D, R: PAD1, HEXABITZ_CONNECTION_PARTS:PAD1
- removed CAN_RX, CAN_TX, CLK, CTS, DIR, IO0, IO1, IO2, IO3, MISO, MOSI, NSS, RTS, RX, SCL, SDA, SWO, TX: PAD4, HEXABITZ_CONNECTION_PARTS:PAD4
- removed JP10, JP2, JP3, JP4, JP5, JP6, JP7, JP8, JP9: (no value), jumper:JP1E
- added VRX, VTX: PAD4, HEXABITZ_CONNECTION_PARTS:PAD4
- added VRX1, VRX2, VRX3, VRX4, VTX1, VTX2, VTX3, VTX4: (no value), jumper:SJ
- JP1: device jumper:JP1E -> pinhead:PINHD-1X2
- P1: value HEXABIT_17.32_NO_P3 -> HEXABIT_17.32_NO_P3_P6_P7_P12; device hexabitz_connectors:HEXABIT_17.32_NO_P3 -> hexabitz_connectors:HEXABIT_17.32_NO_P3_P6_P7_P12
- SWD: device con-lsta:FE05-1 -> con-lstb:MA03-1
Connections:
- removed net N$11: CAN_RX.P$1, U1.BRIDGE_CAN_RX
- removed net N$12: CAN_TX.P$1, U1.BRIDGE_CAN_TX
- removed net N$14: MISO.P$1, U1.BRIDGE_SPI_MISO
- removed net N$15: MOSI.P$1, U1.BRIDGE_SPI_MOSI
- removed net N$16: NSS.P$1, U1.BRIDGE_SPI_NSS
- removed net N$17: CLK.P$1, U1.BRIDGE_SPI_CLK
- removed net N$18: IO0.P$1, U1.BRIDGE_GPIO0
- removed net N$19: IO1.P$1, U1.BRIDGE_GPIO1
- removed net N$20: IO2.P$1, U1.BRIDGE_GPIO2
- removed net N$21: IO3.P$1, U1.BRIDGE_GPIO3
- removed net N$4: SWO.P$1, U1.T_JTDO/T_SWO
- removed net N$5: DIR.P$1, U1.T_SW_DIR
- removed net N$6: RX.P$1, U1.BRIDGE_UART_RX
- removed net N$7: CTS.P$1, U1.BRIDGE_UART_CTS
- removed net N$8: RTS.P$1, U1.BRIDGE_UART_RTS
- removed net N$9: TX.P$1, U1.BRIDGE_UART_TX
- removed net UART5_RX: JP10.2, P1.SD6
- removed net UART5_TX: JP5.2, P1.SU6
- net GND: now also JP1.1; no longer P1.GND1, P1.GND6, SWD.1
- net N$10: no longer SCL.P$1
- net N$13: no longer SDA.P$1
- net SWD_C: now also SWD.2; no longer C.P$1, SWD.4
- net SWD_D: now also SWD.1; no longer D.P$1, SWD.3
- net SWD_R: now also SWD.3; no longer R.P$1, SWD.5
- net UART2_RX: now also VRX1.1; no longer JP6.2
- net UART2_TX: now also VTX1.1; no longer JP1.2
- net UART3_RX: now also VRX3.1; no longer JP8.2
- net UART3_TX: now also VTX3.1; no longer JP3.2
- net UART4_RX: now also VRX4.1; no longer JP9.2
- net UART4_TX: now also VTX4.1; no longer JP4.2
- net UART6_RX: now also VRX2.1; no longer JP7.2
- net UART6_TX: now also VTX2.1; no longer JP2.2
- net VCP_RX: now also VRX.P$1, VRX1.2, VRX2.2, VRX3.2, VRX4.2; no longer JP10.1
- net VCP_TX: now also VTX.P$1, VTX1.2, VTX2.2, VTX3.2, VTX4.2; no longer JP1.1, JP2.1, JP3.1, JP4.1, JP5.1
- net VDD: now also JP1.2; no longer P1.VDD1, P1.VDD6, SWD.2
Other:
- moved on the sheet: R1, R2

Commit message: Generate output files Release V0
Parts:
- R1, R2: value (none) -> 680
Changed lines of the file:
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@@
 <part name="SUPPLY5" library="supply2" library_urn="urn:adsk.eagle:library:372" deviceset="GND" device=""/>
 <part name="SUPPLY6" library="supply2" library_urn="urn:adsk.eagle:library:372" deviceset="GND" device=""/>
-<part name="R1" library="HEXABITZ_RCLS" library_urn="urn:adsk.eagle:library:20064561" deviceset="R-0603" device="" package3d_urn="urn:adsk.eagle:package:1435818/3">
+<part name="R1" library="HEXABITZ_RCLS" library_urn="urn:adsk.eagle:library:20064561" deviceset="R-0603" device="" package3d_urn="urn:adsk.eagle:package:1435818/3" value="680">
 <attribute name="MFN" value="Yageo"/>
 <attribute name="MPN" value="RC0603JR-07680RL"/>
@@
 <attribute name="TOLERANCE" value="5%"/>
 </part>
-<part name="R2" library="HEXABITZ_RCLS" library_urn="urn:adsk.eagle:library:20064561" deviceset="R-0603" device="" package3d_urn="urn:adsk.eagle:package:1435818/3">
+<part name="R2" library="HEXABITZ_RCLS" library_urn="urn:adsk.eagle:library:20064561" deviceset="R-0603" device="" package3d_urn="urn:adsk.eagle:package:1435818/3" value="680">
 <attribute name="MFN" value="Yageo"/>
 <attribute name="MPN" value="RC0603JR-07680RL"/>
@@
 <attribute name="NAME" x="233.4514" y="137.16" size="1.778" layer="95" rot="R90"/>
 <attribute name="VALUE" x="238.252" y="137.16" size="1.778" layer="96" rot="R90"/>
-<attribute name="RESISTANCE" x="233.68" y="143.51" size="1.778" layer="96" rot="R90"/>
 </instance>
 <instance part="R2" gate="G$1" x="118.11" y="125.73" smashed="yes" rot="R180">
-<attribute name="NAME" x="121.92" y="124.2314" size="1.778" layer="95" rot="R180"/>
-<attribute name="VALUE" x="121.92" y="129.032" size="1.778" layer="96" rot="R180"/>
-<attribute name="RESISTANCE" x="115.57" y="124.46" size="1.778" layer="96" rot="R180"/>
+<attribute name="NAME" x="115.57" y="129.3114" size="1.778" layer="95" rot="R180"/>
+<attribute name="VALUE" x="124.46" y="129.032" size="1.778" layer="96" rot="R180"/>
 </instance>
 <instance part="SUPPLY3" gate="G$1" x="106.68" y="130.81" smashed="yes">
